Commit message: [Update][*]增加天工的sim2sim[*]部署天工的跳跃学习

File: resources/robots/tiangong/urdf/tiangong_chz.urdf (robot description, URDF)
Before this commit: robot humanoid, 22 links, 21 joints
Links:
- removed link ankle_pitch_l_link
- removed link ankle_pitch_r_link
- removed link ankle_roll_l_link
- removed link ankle_roll_r_link
- removed link hip_pitch_l_link
- removed link hip_pitch_r_link
- removed link hip_roll_l_link
- removed link hip_roll_r_link
- removed link hip_yaw_l_link
- removed link hip_yaw_r_link
- removed link knee_pitch_l_link
- removed link knee_pitch_r_link
- added link lankle_pitch_link, mass 0.15163; visual mesh filename=../meshes/ankle_pitch_l_link.STL
- added link lankle_roll_link, mass 0.658333536719065; collision mesh filename=../meshes/ankle_roll_l_link.STL; visual mesh filename=../meshes/ankle_roll_l_link.STL
- added link lhip_pitch_link, mass 3.37311; visual mesh filename=../meshes/hip_pitch_l_link.STL
- added link lhip_roll_link, mass 1.12809; visual mesh filename=../meshes/hip_roll_l_link.STL
- added link lhip_yaw_link, mass 1.91605; visual mesh filename=../meshes/hip_yaw_l_link.STL
- added link lknee_pitch_link, mass 2.28832; visual mesh filename=../meshes/knee_pitch_l_link.STL
- added link rankle_pitch_link, mass 0.15163; visual mesh filename=../meshes/ankle_pitch_r_link.STL
- added link rankle_roll_link, mass 0.658333536719064; collision mesh filename=../meshes/ankle_roll_r_link.STL; visual mesh filename=../meshes/ankle_roll_r_link.STL
- added link rhip_pitch_link, mass 3.37311; visual mesh filename=../meshes/hip_pitch_r_link.STL
- added link rhip_roll_link, mass 1.12809; visual mesh filename=../meshes/hip_roll_r_link.STL
- added link rhip_yaw_link, mass 1.91605; visual mesh filename=../meshes/hip_yaw_r_link.STL
- added link rknee_pitch_link, mass 2.28832; visual mesh filename=../meshes/knee_pitch_r_link.STL
- link elbow_l_link: geometry visual mesh filename=../meshes/elbow_l_link.STL
- link elbow_r_link: geometry visual mesh filename=../meshes/elbow_r_link.STL
- link pelvis: geometry collision cylinder length=0.05 radius=0.08; visual mesh filename=../meshes/pelvis.STL
- link shoulder_pitch_l_link: geometry visual mesh filename=../meshes/shoulder_pitch_l_link.STL
- link shoulder_pitch_r_link: geometry visual mesh filename=../meshes/shoulder_pitch_r_link.STL
- link shoulder_roll_l_link: geometry visual mesh filename=../meshes/shoulder_roll_l_link.STL
- link shoulder_roll_r_link: geometry visual mesh filename=../meshes/shoulder_roll_r_link.STL
- link shoulder_yaw_l_link: geometry visual mesh filename=../meshes/shoulder_yaw_l_link.STL
- link shoulder_yaw_r_link: geometry visual mesh filename=../meshes/shoulder_yaw_r_link.STL
- link waist_link: geometry visual mesh filename=../meshes/waist_link.STL
Joints:
- removed joint ankle_pitch_l_joint
- removed joint ankle_pitch_r_joint
- removed joint ankle_roll_l_joint
- removed joint ankle_roll_r_joint
- removed joint hip_pitch_l_joint
- removed joint hip_pitch_r_joint
- removed joint hip_roll_l_joint
- removed joint hip_roll_r_joint
- removed joint hip_yaw_l_joint
- removed joint hip_yaw_r_joint
- removed joint knee_pitch_l_joint
- removed joint knee_pitch_r_joint
- removed joint shoulder_pitch_l_joint
- removed joint shoulder_pitch_r_joint
- added joint lankle_pitch_joint: type revolute, parent lknee_pitch_link, child lankle_pitch_link, origin xyz=0 0 -0.3 rpy=0 0 0, axis 0 1 0, limit lower=-1.22 upper=0.5236 effort=60 velocity=7.8
- added joint lankle_roll_joint: type revolute, parent lankle_pitch_link, child lankle_roll_link, origin xyz=0 0 0 rpy=0 0 0, axis 1 0 0, limit lower=-0.4363 upper=0.4363 effort=30 velocity=7.8
- added joint lhip_pitch_joint: type revolute, parent lhip_yaw_link, child lhip_pitch_link, origin xyz=0 0 0 rpy=0 0 0, axis 0 1 0, limit lower=-1.57 upper=0.5236 effort=150 velocity=12
- added joint lhip_roll_joint: type revolute, parent pelvis, child lhip_roll_link, origin xyz=0 0.13 -0.0659230484541305 rpy=0 0 0, axis 1 0 0, limit lower=-0.97 upper=0.97 effort=150 velocity=12
- added joint lhip_yaw_joint: type revolute, parent lhip_roll_link, child lhip_yaw_link, origin xyz=0 0 -0.116 rpy=0 0 0, axis 0 0 1, limit lower=-1.0472 upper=1.0472 effort=90 velocity=14
- added joint lknee_pitch_joint: type revolute, parent lhip_pitch_link, child lknee_pitch_link, origin xyz=0 0 -0.3 rpy=0 0 0, axis 0 1 0, limit lower=0.1745 upper=2.443 effort=150 velocity=12
- added joint lshoulder_pitch_joint: type revolute, parent waist_link, child shoulder_pitch_l_link, origin xyz=0 0.17581 0.43652 rpy=0.2618 0 0, axis 0 1 0, limit lower=-3.14 upper=0.97 effort=36 velocity=7.8
- added joint rankle_pitch_joint: type revolute, parent rknee_pitch_link, child rankle_pitch_link, origin xyz=0 0 -0.3 rpy=0 0 0, axis 0 1 0, limit lower=-1.22 upper=0.5236 effort=60 velocity=7.8
- added joint rankle_roll_joint: type revolute, parent rankle_pitch_link, child rankle_roll_link, origin xyz=0 0 0 rpy=0 0 0, axis 1 0 0, limit lower=-0.4363 upper=0.4363 effort=30 velocity=7.8
- added joint rhip_pitch_joint: type revolute, parent rhip_yaw_link, child rhip_pitch_link, origin xyz=0 0 0 rpy=0 0 0, axis 0 1 0, limit lower=-1.57 upper=0.5236 effort=150 velocity=12
- added joint rhip_roll_joint: type revolute, parent pelvis, child rhip_roll_link, origin xyz=0 -0.13 -0.0659230484541306 rpy=0 0 0, axis 1 0 0, limit lower=-0.97 upper=0.97 effort=150 velocity=12
- added joint rhip_yaw_joint: type revolute, parent rhip_roll_link, child rhip_yaw_link, origin xyz=0 0 -0.116 rpy=0 0 0, axis 0 0 1, limit lower=-1.0472 upper=1.0472 effort=90 velocity=14
- added joint rknee_pitch_joint: type revolute, parent rhip_pitch_link, child rknee_pitch_link, origin xyz=0 0 -0.3 rpy=0 0 0, axis 0 1 0, limit lower=0.1745 upper=2.443 effort=150 velocity=12
- added joint rshoulder_pitch_joint: type revolute, parent waist_link, child shoulder_pitch_r_link, origin xyz=0 -0.17577 0.43652 rpy=-0.2618 0 0, axis 0 1 0, limit lower=-3.14 upper=0.97 effort=36 velocity=7.8
